File: Aeroq Hardware/Aeroq Hardware.kicad_sch (KiCad schematic)
At the start: 0 parts

Commit message: schematic and pcb initial
Parts:
- added C1, C6, C9: 10uf/25V, Capacitor_SMD:C_0603_1608Metric, symbol Device:C
- added C10, C12, C13, C14, C16, C17, C18, C19, C23, C24: 4.7uf/25V, Capacitor_SMD:C_0603_1608Metric, symbol Device:C
- added C11, C15, C2, C3, C5, C7, C8: 0.1uf/50V, Capacitor_SMD:C_0603_1608Metric, symbol Device:C
- added C20, C21, C22, C25, C4: 1uf/50V, Capacitor_SMD:C_0603_1608Metric, symbol Device:C
- added D1, D5: 1N5819WS, Diode_SMD:D_SOD-323, symbol Diode:1N5819WS
- added D10, D11, D12: MBR0530, Diode_SMD:D_SOD-123, symbol Diode:MBR0530
- added D2, D3, D4, D6, D7, D8: LESD5D5.0CT1G, custom_footprints:TVS_LESD5D5.0CT1G, symbol LESD5D5.0CT1G:LESD5D5.0CT1G
- added D9: LED, LED_SMD:LED_0603_1608Metric, symbol Device:LED
- added FPC1: ~, Library:FPC-SMD_24P-P0.50_FPC-05FB-24PH20, symbol FPC-05FB-24PH20:FPC-05FB-24PH20
- added J1: USB_C_Receptacle_USB2.0_16P, USBC_SMD_VERTICAL:TYPE-C-SMD_USB4120-03-C, symbol Connector:USB_C_Receptacle_USB2.0_16P
- added J2: Conn_01x05, Connector_JST:JST_PH_S5B-PH-K_1x05_P2.00mm_Horizontal, symbol Connector_Generic:Conn_01x05
- added L1: 10uH/1A, Inductor_SMD:L_1210_3225Metric, symbol Device:L
- added Q1: Si1308EDL, Package_TO_SOT_SMD:SOT-323_SC-70, symbol Transistor_FET:Si1308EDL
- added R1, R10, R11, R3, R6, R7, R8: 10kR, Resistor_SMD:R_0402_1005Metric, symbol Device:R
- added R100, R200, R4, R5: 5kR, Resistor_SMD:R_0402_1005Metric, symbol Device:R
- added R12: 0.47R, Resistor_SMD:R_0402_1005Metric, symbol Device:R
- added R9: 3R, Resistor_SMD:R_0402_1005Metric, symbol Device:R
- added S1, S2: TS-1187A-B-A-B, custom_footprints:SW_TS-1187A-B-A-B, symbol TS-1187A-B-A-B:TS-1187A-B-A-B
- added TP1, TP10, TP11, TP2, TP3, TP4, TP5, TP6, TP7, TP8, TP9: TestPoint, TestPoint:TestPoint_Pad_D1.5mm, symbol Connector:TestPoint
- added U1: ~, USBC_SMD_VERTICAL:TYPE-C-SMD_USB4120-03-C, symbol TYPE-C 16PLT-H10:TYPE-C 16PLT-H10.0
- added U2: ESP32-C3-MINI-1-N4, custom_footprints:XCVR_ESP32-C3-MINI-1-N4, symbol ESP32-C3-MINI-1-N4:ESP32-C3-MINI-1-N4
- added U3: AMS1117-3.3, Package_TO_SOT_SMD:SOT-223-3_TabPin2, symbol Regulator_Linear:AMS1117-3.3
- added U4: SCD40-D-R1, Sensor:Sensirion_SCD4x-1EP_10.1x10.1mm_P1.25mm_EP4.8x4.8mm, symbol SCD40-D-R1:SCD40-D-R1
Connections:
- new net: C22.1, FPC1.19
- new net: C12.2, FPC1.4
- new net: C17.2, D12.2 (A), L1.2, Q1.3 (D)
- new net: R4.2, U1.B5 (CC2)
- new net: C14.2, FPC1.5
- new net: R5.2, U1.A5 (CC1)
- new net: FPC1.8, R10.1, R9.1
- new net: D9.2 (A), R6.1
- new net: C21.1, FPC1.18
- new net: C17.1, D10.1 (K), D11.2 (A)
- new net: C20.2, FPC1.16
- new net: C24.2, FPC1.22
- new net: C23.2, FPC1.20
- new net: J1.A5 (CC1), R200.2
- new net: U2.10 (NC), U2.15 (NC), U2.17 (NC), U2.24 (NC), U2.25 (NC), U2.28 (NC), U2.29 (NC), U2.32 (NC), U2.33 (NC), U2.34 (NC), U2.35 (NC), U2.4 (NC), U2.7 (NC), U2.9 (NC)
- new net: J1.B5 (CC2), R100.2
- new net: C25.2, FPC1.24
- new net: U4.1 (DNC), U4.11 (DNC), U4.12 (DNC), U4.13 (DNC), U4.14 (DNC), U4.15 (DNC), U4.16 (DNC), U4.17 (DNC), U4.18 (DNC), U4.2 (DNC), U4.3 (DNC), U4.4 (DNC), U4.5 (DNC), U4.8 (DNC)
- new net +3.3V: C1.2, C15.1, C16.2, C18.1, C2.1, C8.1, C9.2, L1.1, R1.2, R10.2, R3.2, R6.2, R7.2, R8.2, TP2.1, U2.3 (3V3), U3.2 (VO), U4.19 (VDDH), U4.7 (VDD)
- new net +5V: C10.2, C11.1, C6.2, C7.1, D1.1 (K), D5.1 (K), J2.1 (Pin_1), TP3.1, U3.3 (VI)
- new net BUSY: FPC1.9, TP10.1, U2.13 (IO1)
- new net CHIP_PU: C4.2, C5.1, R1.1, S2.C, S2.D, U2.8 (EN)
- new net CS: FPC1.12, TP8.1, U2.19 (IO5)
- new net D+: D4.2, D8.2, J1.A6 (D+), J1.B6 (D+), U1.A6 (DP1), U1.B6 (DP2), U2.26 (IO18)
- new net D-: D3.2, D7.2, J1.A7 (D-), J1.B7 (D-), U1.A7 (DN1), U1.B7 (DN2), U2.27 (IO19)
- new net DC: FPC1.11, TP11.1, U2.18 (IO4)
- new net GDR: FPC1.2, Q1.1 (G), R11.2
- new net GND: C1.1, C10.1, C11.2, C12.1, C13.2, C14.1, C15.2, C16.1, C18.2, C19.2, C2.2, C20.1, C21.2, C22.2, C23.1, C24.1, C25.1, C3.2, C4.1, C5.2, C6.1, C7.2, C8.2, C9.1, D11.1 (K), D2.1, D3.1, D4.1, D6.1, D7.1, D8.1, D9.1 (K), FPC1.17, FPC1.25, FPC1.26, J1.A1 (GND), J1.A12 (GND), J1.B1 (GND), J1.B12 (GND), J1.S1 (SHIELD), J2.2 (Pin_2), J2.5 (Pin_5), R100.1, R11.1, R12.1, R200.1, R4.1, R5.1, R9.2, S1.A, S1.B, S2.A, S2.B, TP1.1, U1.A1 (GND), U1.A12 (GND), U1.B1 (GND), U1.B12 (GND), U2.1 (GND), U2.11 (GND), U2.14 (GND), U2.2 (GND), U2.36 (GND), U2.37 (GND), U2.38 (GND), U2.39 (GND), U2.40 (GND), U2.41 (GND), U2.42 (GND), U2.43 (GND), U2.44 (GND), U2.45 (GND), U2.46 (GND), U2.47 (GND), U2.48 (GND), U2.49_1 (GND), U2.49_2 (GND), U2.49_3 (GND), U2.49_4 (GND), U2.49_5 (GND), U2.49_6 (GND), U2.49_7 (GND), U2.49_8 (GND), U2.49_9 (GND), U2.50 (GND), U2.51 (GND), U2.52 (GND), U2.53 (GND), U3.1 (GND), U4.20 (GND), U4.21 (GND), U4.6 (GND)
- new net GPIO2: R3.1, U2.5 (IO2)
- new net GPIO9: C3.1, S1.C, S1.D, U2.23 (IO9)
- new net PREVGH: C19.1, D12.1 (K), FPC1.21
- new net PREVGL: C13.1, D10.2 (A), FPC1.23
- new net RES: FPC1.10, TP9.1, U2.6 (IO3)
- new net RESE: FPC1.3, Q1.2 (S), R12.2
- new net SCL: J2.4 (Pin_4), R7.1, TP4.1, U2.12 (IO0), U4.9 (SCL)
- new net SCLK: FPC1.13, TP7.1, U2.20 (IO6)
- new net SDA: J2.3 (Pin_3), R8.1, TP5.1, U2.22 (IO8), U4.10 (SDA)
- new net SDI: FPC1.14, TP6.1, U2.21 (IO7)
- new net VBUS: D1.2 (A), D2.2, D5.2 (A), D6.2, J1.A4 (VBUS), J1.A9 (VBUS), J1.B4 (VBUS), J1.B9 (VBUS), U1.A4 (VBUS), U1.A9 (VBUS), U1.B4 (VBUS), U1.B9 (VBUS)
- no-connect marks 0 -> 13
