File: Aeroq Hardware/v3/Aeroq Hardware v3.kicad_pcb (KiCad board)
At the start: 2 copper layers, 45 x 45 mm, 56 parts, among them Q1 Si1308EDL, U2 ESP32-C3-MINI-1-N4, U3 AMS1117-3.3, U4 SCD40-D-R1

Commit message: updates to kicad schematic/pcb
Parts:
- removed CN1: ~, CONN-SMD_5P-P2.00_ZX-PH2.0-WT5P:CONN-SMD_5P-P2.00_ZX-PH2.0-WT5P
- added U5: ~, JST SM05B-GHS-TB(LF)(SN):CONN-SMD_5P-P1.25_SM05B-GHS-TB-LF-SN, F.Cu at (124.8, 77.8)
- moved C22 1.13 mm to (96.7, 89.6)
- moved C21 1.04 mm to (96.7, 91.5)
- moved C23 0.96 mm to (96.7, 87.5)
- moved C20 0.94 mm to (96.1, 93.9)
- moved TP5 0.75 mm to (112.0, 95.9)
- renumbered GND to TP1, 3.3V to TP2, 5V to TP3, SCL to TP4, SDA to TP5
Connections:
- C20 pad 2: Net-(C20-Pad2) -> +3.3V
- FPC1 pad 15: unconnected-(FPC1-Pad15) -> +3.3V
- FPC1 pad 16: Net-(C20-Pad2) -> +3.3V
- U2 pad 26: D+ -> D-
- U2 pad 27: D- -> D+
Routing:
- net +3.3V: track 175.6 -> 213.7 mm, vias 6 -> 8
- net +5V: track 40.7 -> 53.7 mm
- net SCL: track 82.3 -> 86.4 mm
- net D-: track 43.8 -> 39.9 mm
- net Net-(C20-Pad2): track 2.96 -> 0.00 mm
- net GND: track 27.5 -> 24.8 mm
- net SDA: track 74.4 -> 76.2 mm
- net D+: track 36.8 -> 38.4 mm
- net Net-(C23-Pad2): track 5.64 -> 6.54 mm
- net Net-(C22-Pad1): track 4.11 -> 4.99 mm
- net VBUS: track 21.4 -> 20.8 mm
Other:
- board text added: "3.3V"
- board text added: "5V"
- board text added: "Aeroq v3"
- board text added: "BOOT"
- board text added: "ESP32-C3"
- board text added: "GND"
- board text added: "RESET"
- board text added: "SCD40"
- board text added: "SCL"
- board text added: "SDA"
- board text added: "SEN54"
- board text added: "USB-C"

Commit message: PCB Updates
Parts:
- D2, D3, D4: footprint SOD-523_L1.2-W0.8-LS1.6-BI:SOD-523_L1.2-W0.8-LS1.6-BI -> Project Footprints:SOD-523_L1.2-W0.8-LS1.6-BI
- FPC1: footprint FPC-SMD_24P-P0.50_FPC-05FB-24PH20:FPC-SMD_24P-P0.50_FPC-05FB-24PH20 -> Project Footprints:FPC-SMD_24P-P0.50_FPC-05FB-24PH20
- SW1, SW2: footprint SW-SMD_L3.9-W3.0-P4.45:SW-SMD_L3.9-W3.0-P4.45 -> Project Footprints:SW-SMD_L3.9-W3.0-P4.45
- U1: footprint USBC_SMD_VERTICAL:TYPE-C-SMD_USB4120-03-C -> Project Footprints:TYPE-C-SMD_USB4120-03-C
- U2: footprint custom_footprints:XCVR_ESP32-C3-MINI-1-N4 -> Project Footprints:XCVR_ESP32-C3-MINI-1-N4
- U4: footprint Sensor:Sensirion_SCD4x-1EP_10.1x10.1mm_P1.25mm_EP4.8x4.8mm -> Project Footprints:XDCR_SCD40-D-R1
Routing:
- net GND: track 24.8 -> 29.8 mm
- net +3.3V: track 213.7 -> 212.5 mm
